Commit message: Added camera support. Can be viewed through rqt

File: uuv_simulator/manta_description/urdf/manta_sensors.xacro (robot description, xacro)
@@ -37,8 +37,9 @@
     <origin xyz="0 0 0" rpy="0 0 0"/>
   </xacro:default_imu_macro>
-  <!-- Mount a camera
+  <!-- Mount a camera -->
   <xacro:default_camera namespace="${namespace}" parent_link="${namespace}/base_link" suffix="">
-    <origin xyz="1.15 0 0.4" rpy="0 0.6 0"/>
+    <origin xyz="0.5 0 0.4" rpy="0 0 0"/>
   </xacro:default_camera>
+  <!--
   <xacro:default_camera namespace="${namespace}" parent_link="${namespace}/base_link" suffix="right">
     <origin xyz="1.15 -0.63 0.4" rpy="0 0.6 0.4"/>

Commit message: moved the position of front camera and changed mass

File: uuv_simulator/manta_description/urdf/manta_sensors.xacro (robot description, xacro)
@@ -39,5 +39,5 @@
   <!-- Mount a camera -->
   <xacro:default_camera namespace="${namespace}" parent_link="${namespace}/base_link" suffix="">
-    <origin xyz="0.5 0 0.4" rpy="0 0 0"/>
+    <origin xyz="0.30 0.0 0." rpy="0 0 0"/>
   </xacro:default_camera>
   <!--

File: uuv_simulator/uuv_sensor_plugins/uuv_sensor_ros_plugins/urdf/camera_snippets.xacro (robot description, xacro)
@@ -28,5 +28,5 @@
       parent_link="${parent_link}"
       topic="camera"
-      mass="0.1"
+      mass="0.001"
       update_rate="30"
       hfov="1.5125"

Commit message: Changed the size of all sensors and included DVL

File: uuv_simulator/manta_description/urdf/manta_sensors.xacro (robot description, xacro)
@@ -13,11 +13,12 @@
 -->
 <robot xmlns:xacro="http://www.ros.org/wiki/xacro">
-  <!-- DVL  ->
+  <!-- DVL -->
   <xacro:default_dvl_macro
     namespace="${namespace}"
     parent_link="${namespace}/base_link"
     inertial_reference_frame="${inertial_reference_frame}">
-    <origin xyz="-1.4 0 -0.312" rpy="0 ${0.5*pi} 0"/>
+    <origin xyz="0 0 0" rpy="0 ${0.5*pi} 0"/>
   </xacro:default_dvl_macro>
+<!--
   <!- Magnetometer  ->
   <xacro:default_magnetometer namespace="${namespace}" parent_link="${namespace}/base_link"/>
@@ -25,6 +26,6 @@
   <xacro:default_rpt namespace="${namespace}" parent_link="${namespace}/base_link">
     <origin xyz="-1.32 0 0.8" rpy="0 0 0"/>
-  </xacro:default_rpt>
-  <!- Pressure  -->
+  </xacro:default_rpt> -->
+  <!-- Pressure  -->
   <xacro:default_pressure_macro namespace="${namespace}" parent_link="${namespace}/base_link">
     <origin xyz="0 0 0" rpy="0 0 0"/>

File: uuv_simulator/uuv_sensor_plugins/uuv_sensor_ros_plugins/urdf/dvl_snippets.xacro (robot description, xacro)
@@ -31,5 +31,5 @@
       noise_sigma="0"
       noise_amplitude="0"
-      scale="1">
+      scale="0.5">
       <xacro:insert_block name="origin" />
     </xacro:dvl_plugin_macro>
@@ -62,5 +62,5 @@
       noise_sigma="0"
       noise_amplitude="0"
-      scale="1">
+      scale="0.5">
       <xacro:insert_block name="origin" />
     </xacro:dvl_plugin_macro>

File: uuv_simulator/uuv_sensor_plugins/uuv_sensor_ros_plugins/urdf/pressure_snippets.xacro (robot description, xacro)
@@ -69,5 +69,5 @@
       <visual>
         <geometry>
-          <mesh filename="file://$(find uuv_sensor_ros_plugins)/meshes/pressure.dae" scale="1 1 1"/>
+          <mesh filename="file://$(find uuv_sensor_ros_plugins)/meshes/pressure.dae" scale="0.1 0.1 0.1"/>
         </geometry>
       </visual>

Commit message: added extra camera facing down

File: uuv_simulator/manta_description/urdf/manta_sensors.xacro (robot description, xacro)
@@ -31,11 +31,11 @@
   </xacro:default_imu_macro>
   <!-- Mount a camera -->
-  <xacro:default_camera namespace="${namespace}" parent_link="${namespace}/base_link" suffix="">
-    <origin xyz="0.30 0.0 0." rpy="0 0 0"/>
+  <xacro:default_camera namespace="${namespace}" parent_link="${namespace}/base_link" suffix="front">
+    <origin xyz="0.29 0.0 0." rpy="0 0 0"/>
   </xacro:default_camera>
-  <!--
-  <xacro:default_camera namespace="${namespace}" parent_link="${namespace}/base_link" suffix="right">
-    <origin xyz="1.15 -0.63 0.4" rpy="0 0.6 0.4"/>
+  <xacro:default_camera namespace="${namespace}" parent_link="${namespace}/base_link" suffix="under">
+    <origin xyz="0.15 0.0 -0.06" rpy="0 ${0.5*pi} 0"/>
   </xacro:default_camera>
+<!--
   <xacro:default_camera namespace="${namespace}" parent_link="${namespace}/base_link" suffix="left">
     <origin xyz="1.15 0.63 0.4" rpy="0 0.6 -0.4"/>
