Commit message: Changed COG and COB for Manta. Also added Collision mesh

File: uuv_simulator/manta_description/urdf/manta_base.xacro (robot description, xacro)
@@ -36,7 +36,7 @@
   <!-- minion_usv_height is not really! It's just for run... We need first calculate the Fossen parameters -->
   <!-- Volume -->
-  <xacro:property name="volume" value="0.01754"/>
+  <xacro:property name="volume" value="0.01854"/>
   <!-- Center of gravity -->
-  <xacro:property name="cog" value="0 0 0"/>
+  <xacro:property name="cog" value="0 0 -0.03"/>
   <!--
   Center of buoyancy according to eq. (3.1) p. 28 in Berg2012.
@@ -44,5 +44,5 @@
   assume NWU (otherwise cob is below cog?). 0.155
   -->
-  <xacro:property name="cob" value="0 0 0"/>
+  <xacro:property name="cob" value="0 0 0.05"/>
   <!-- Fluid density -->
   <xacro:property name="rho" value="1028"/>
@@ -83,11 +83,10 @@
           </geometry>
         </visual>
-        <!-- In rexrov2_base they made collision planes to minize the GPU load -->
-        <!-- <collision>
-          <origin xyz="0 0 0" rpy="0 0 0"/>
-          <geometry>
-            <mesh filename="${collision_mesh_file}" scale="1 1 1" />
-          </geometry>
-        </collision> -->
+        <!-- In manta_base i've made collision planes to minize the GPU load -->
+    <collision>
+      <geometry>
+        <box size="0.3 03 0.15"/>
+      </geometry>
+    </collision>
       </link>
     <gazebo reference="${namespace}/base_link">

Commit message: changed color of manta base and actuators. Changed collision mesh

File: uuv_simulator/manta_description/urdf/manta_base.xacro (robot description, xacro)
@@ -22,5 +22,5 @@
   -->
   <!-- Mass -->
-  <xacro:property name="mass" value="18"/>
+  <xacro:property name="mass" value="19.0"/>
   <!-- Describing the dimensions of the vehicle's bounding box: width, length, height -->
   <xacro:property name="x_size" value="0.448"/>
@@ -51,5 +51,5 @@
   <xacro:macro name="manta_base" params="namespace *gazebo inertial_reference_frame">
    <!-- Rigid body description of the base link -->
-      <link name="${namespace}/base_link">
+    <link name="${namespace}/base_link">
         <!--
           Be careful to setup the coefficients for the inertial tensor,
@@ -77,9 +77,10 @@
         <!-- In manta_base i've made collision planes to minize the GPU load -->
     <collision>
+      <origin xyz="0 0 ${0}" rpy="0 0 0"/>
       <geometry>
-        <box size="0.3 03 0.15"/>
+        <sphere radius="${0.25}"/>
       </geometry>
     </collision>
-      </link>
+  </link>
     <gazebo reference="${namespace}/base_link">
       <selfCollide>false</selfCollide>
@@ -100,3 +101,6 @@
   <xacro:include filename="$(find manta_description)/urdf/manta_sensors.xacro"/>
   </xacro:macro>
+  <gazebo reference="${namespace}/base_link">
+    <material>Gazebo/FlatBlack</material>
+  </gazebo>
 </robot>

File: uuv_simulator/uuv_gazebo_plugins/uuv_gazebo_ros_plugins/urdf/thruster_snippets.xacro (robot description, xacro)
@@ -110,6 +110,8 @@
       </plugin>
     </gazebo>
+   <!-- Choose thruster color -->
     <gazebo reference="${namespace}/thruster_${thruster_id}">
       <selfCollide>false</selfCollide>
+    <material>Gazebo/Red</material>
     </gazebo>
   </xacro:macro>

File: uuv_simulator/uuv_sensor_plugins/uuv_sensor_ros_plugins/urdf/magnetometer_snippets.xacro (robot description, xacro)
@@ -54,5 +54,5 @@
       <visual>
         <geometry>
-          <box size="0.1 0.1 0.1" />
+          <box size="0.05 0.05 0.05" />
         </geometry>
       </visual>

Commit message: changed inertia for manta

File: uuv_simulator/manta_description/urdf/manta_base.xacro (robot description, xacro)
@@ -59,8 +59,9 @@
           <mass value="${mass}" />
           <origin xyz="${cog}" rpy="0 0 0"/>
-          <!-- <inertia ixx="525.39" ixy="1.44" ixz="33.41" iyy="794.20" iyz="2.6" izz="691.23"/> -->
+           <!-- ixx="${0.80947}" ixy="-0.00308" ixz="-0.01546"
+            iyy="${0.87794}" iyz="0.06283" izz="${1.57147}" />  -->
           <inertia
-            ixx="${0.80947}" ixy="-0.00308" ixz="-0.01546"
-            iyy="${0.87794}" iyz="0.06283" izz="${1.57147}" />
+            ixx="${0.503217}" ixy="${0.000204}" ixz="${-0.000526}"
+            iyy="${0.493449}" iyz="${0.000038}" izz="${0.919819}" />
         </inertial>
         <!-- This visual geometry representation can be used when running
