Commit message: new thrusters added to the simulator

File: uuv_simulator/manta_description/urdf/manta_actuators.xacro (robot description, xacro)
@@ -42,5 +42,5 @@
   </xacro:thruster_macro>
   <xacro:thruster_macro namespace="${namespace}" thruster_id="4"> <!-- lat back left-->
-    <origin xyz="-0.12070 0.12070 0" rpy="${0*d2r} ${0*d2r} ${45*d2r}"/>
+    <origin xyz="-0.20506 0.20506 0" rpy="${0*d2r} ${0*d2r} ${45*d2r}"/>
   </xacro:thruster_macro>
   <xacro:thruster_macro namespace="${namespace}" thruster_id="5"> <!-- lat back right -->

Commit message: Added new propellers and updated the hydrodynamic coeff of Manta in simulator

File: uuv_simulator/manta_description/urdf/manta_actuators.xacro (robot description, xacro)
@@ -15,5 +15,6 @@
 <!-- Here you can put in whatever kind of model you want and it will
   still function as a propeller                                      -->
-  <xacro:property name="prop_mesh_file" value="file://$(find manta_description)/mesh/prop.dae"/>
+  <xacro:property name="prop_mesh_file_cw" value="file://$(find manta_description)/mesh/t200_propccw.dae"/>
+  <xacro:property name="prop_mesh_file_ccw" value="file://$(find manta_description)/mesh/t200_propcw.dae"/>
   <!-- <xacro:property name="prop_mesh_file" value="file://$(find manta_description)/mesh/manipulator_claw.dae"/> -->
   <!-- Thruster joint and link snippet -->
@@ -23,22 +24,42 @@
       namespace="${namespace}"
       thruster_id="${thruster_id}"
-      mesh_filename="${prop_mesh_file}"
+      mesh_filename="${prop_mesh_file_cw}"
       dyn_time_constant="0.05"
-      rotor_constant="0.00031">
+      rotor_constant="0.0031">
       <xacro:insert_block name="origin"/>
     </xacro:thruster_module_first_order_basic_fcn_macro>
   </xacro:macro>
+  <xacro:macro name="thruster_macro_ccw"
+    params="namespace thruster_id *origin">
+    <xacro:thruster_module_first_order_basic_fcn_macro
+      namespace="${namespace}"
+      thruster_id="${thruster_id}"
+      mesh_filename="${prop_mesh_file_ccw}"
+      dyn_time_constant="0.05"
+      rotor_constant="0.0031">
+      <xacro:insert_block name="origin"/>
+    </xacro:thruster_module_first_order_basic_fcn_macro>
+  </xacro:macro>
+<!-- Top thrusters -->
   <xacro:thruster_macro namespace="${namespace}" thruster_id="0"> <!-- heave back left prop up-->
-  <origin xyz="-0.12070 0.12070 0" rpy="${0*d2r} ${-74.53*d2r} ${-53.21*d2r}"/>
+  <origin xyz="-0.12070 0.12070 0" rpy="0 -1.5707963268 0"/>
   </xacro:thruster_macro>
   <xacro:thruster_macro namespace="${namespace}" thruster_id="1"> <!-- heave bacl right prop up-->
-    <origin xyz="-0.12070 -0.12070 0" rpy="${0*d2r} ${-74.53*d2r} ${53.21*d2r}"/>
+    <origin xyz="-0.12070 -0.12070 0" rpy="0 -1.5707963268 0"/>
   </xacro:thruster_macro>
   <xacro:thruster_macro namespace="${namespace}" thruster_id="2"> <!-- heave front left prop up-->
-    <origin xyz="0.12070 0.12070 0" rpy="${0*d2r} ${-105.47*d2r} ${53.21*d2r}"/>
+    <origin xyz="0.12070 0.12070 0" rpy="0 -1.5707963268 0"/>
   </xacro:thruster_macro>
   <xacro:thruster_macro namespace="${namespace}" thruster_id="3"> <!-- heave front right prop up-->
-    <origin xyz="0.12070 -0.12070 0" rpy="${0*d2r} ${-105.47*d2r} ${-53.21*d2r}"/>
+    <origin xyz="0.12070 -0.12070 0" rpy="0 -1.5707963268 0"/>
   </xacro:thruster_macro>
+ <!-- Front thrusters -->
+  <xacro:thruster_macro namespace="${namespace}" thruster_id="6"> <!-- lat front left-->
+    <origin xyz="0.20506 0.20506 0" rpy="${0*d2r} ${0*d2r} ${135*d2r}"/>
+  </xacro:thruster_macro>
+  <xacro:thruster_macro namespace="${namespace}" thruster_id="7"> <!-- lat front right -->
+    <origin xyz="0.20506 -0.20506 0" rpy="${0*d2r} ${0*d2r} ${-135*d2r}"/>
+  </xacro:thruster_macro>
+ <!-- Back thrusters -->
   <xacro:thruster_macro namespace="${namespace}" thruster_id="4"> <!-- lat back left-->
     <origin xyz="-0.20506 0.20506 0" rpy="${0*d2r} ${0*d2r} ${45*d2r}"/>
@@ -47,9 +68,3 @@
     <origin xyz="-0.20506 -0.20506 0" rpy="${0*d2r} ${0*d2r} ${-45*d2r}"/>
   </xacro:thruster_macro>
-  <xacro:thruster_macro namespace="${namespace}" thruster_id="6"> <!-- lat front left-->
-    <origin xyz="0.20506 0.20506 0" rpy="${0*d2r} ${0*d2r} ${135*d2r}"/>
-  </xacro:thruster_macro>
-  <xacro:thruster_macro namespace="${namespace}" thruster_id="7"> <!-- lat front right -->
-    <origin xyz="0.20506 -0.20506 0" rpy="${0*d2r} ${0*d2r} ${-135*d2r}"/>
-  </xacro:thruster_macro>
 </robot>

File: uuv_simulator/manta_description/urdf/manta_base.xacro (robot description, xacro)
@@ -25,54 +25,75 @@
   <xacro:include filename="$(find uuv_sensor_ros_plugins)/urdf/sensor_snippets.xacro"/>
   <xacro:include filename="$(find uuv_gazebo_ros_plugins)/urdf/snippets.xacro"/>
+<!--
+    Vehicle's parameters (remember to enter the model parameters below)
+  -->
+  <!-- Mass -->
+  <xacro:property name="mass" value="18"/>
+  <!-- Describing the dimensions of the vehicle's bounding box: width, length, height -->
+  <xacro:property name="x_size" value="0.448"/>
+  <xacro:property name="y_size" value="0.444"/>
+  <xacro:property name="z_size" value="0.28066"/>
+  <!-- minion_usv_height is not really! It's just for run... We need first calculate the Fossen parameters -->
+  <!-- Volume -->
+  <xacro:property name="volume" value="0.01754"/>
+  <!-- Center of gravity -->
+  <xacro:property name="cog" value="0 0 0"/>
+  <!--
+  Center of buoyancy according to eq. (3.1) p. 28 in Berg2012.
+  The original values, [0.0822, -0.00773, 0.3872] however, seem to
+  assume NWU (otherwise cob is below cog?). 0.155
+  -->
+  <xacro:property name="cob" value="0 0 0"/>
+  <!-- Fluid density -->
+  <xacro:property name="rho" value="1028"/>
+  <!--
+    Visual mesh file for the vehicle, usually in DAE (Collada) format. Be sure to store the
+    mesh with the origin of the mesh on the same position of the center of mass, otherwise
+    the mesh pose will have to be corrected below in the <visual> block.
+    Open the meshes for the RexROV vehicle in Blender to see an example on the mesh placement.
+  -->
   <!-- Parameters -->
   <xacro:property name="namespace" value="manta"/>
   <xacro:property name="visual_mesh_file" value="file://$(find manta_description)/mesh/manta_shell.dae"/>
-  <xacro:property name="prop_mesh_file" value="file://$(find manta_description)/mesh/prop.dae"/>
-  <!-- Mass, see p.28 in Berg2012 -->
-  <xacro:property name="mass" value="1600.0"/>
   <xacro:macro name="manta_base" params="namespace *gazebo inertial_reference_frame">
-    <!-- base_link according to ROS conventions: x forward, z up -->
-    <link name="${namespace}/base_link">
-      <inertial>
-        <mass value="${mass}"/>
-        <origin xyz="0 0 0"/>
-        <inertia ixx="525.39" ixy="1.44" ixz="33.41" iyy="794.20" iyz="2.6" izz="691.23"/>
-      </inertial>
-      <visual>
-        <origin xyz="0 0 0" rpy="0 0 0"/>
-        <geometry>
-          <mesh filename="${visual_mesh_file}" scale="1 1 1"/>
-        </geometry>
-      </visual>
-      <!-- bottom plate -->
-      <collision>
-        <origin xyz="0 0 -0.75" rpy="0 0 0"/>
-        <geometry>
-          <box size="2.56 1.50 0.10"/>
-        </geometry>
-      </collision>
-      <!-- top plate -->
-      <collision>
-        <origin xyz="0 0 0.60" rpy="0 0 0"/>
-        <geometry><box size="2.56 1.50 0.40"/></geometry>
-      </collision>
-      <!-- left / right sides -->
-      <collision>
-        <origin xyz="-0.20 0.70 -0.15" rpy="0 0 0"/>
-        <geometry><box size="2.20 0.10 1.10"/></geometry>
-      </collision>
-      <collision>
-        <origin xyz="-0.20 -0.70 -0.15" rpy="0 0 0"/>
-        <geometry><box size="2.20 0.10 1.10"/></geometry>
-      </collision>
-    </link>
+   <!-- Rigid body description of the base link -->
+      <link name="${namespace}/base_link">
+        <!--
+          Be careful to setup the coefficients for the inertial tensor,
+          otherwise your model will become unstable on Gazebo
+        -->
+        <inertial>
+          <mass value="${mass}" />
+          <origin xyz="${cog}" rpy="0 0 0"/>
+          <!-- <inertia ixx="525.39" ixy="1.44" ixz="33.41" iyy="794.20" iyz="2.6" izz="691.23"/> -->
+          <inertia
+            ixx="${0.6*mass*y_size*y_size + 0.6*mass*z_size*z_size}" ixy="0.0" ixz="0.0"
+            iyy="${0.6*mass*x_size*x_size + 0.6*mass*z_size*z_size}" iyz="0.0"
+            izz="${0.001*mass*x_size*x_size + 0.001*mass*y_size*y_size}" />
+        </inertial>
+        <!-- This visual geometry representation can be used when running
+             tasks in which you need Gazebo to start quickly
+        -->
+        <!-- <xacro:if value="${use_simplified_mesh}"> -->
+        <!-- Code in rexrov2_base.xacro if use the flag use_simplified_mesh -->
+        <visual>
+          <origin xyz="0 0 0" rpy="0 0 0"/>
+          <geometry>
+            <mesh filename="${visual_mesh_file}" scale="1 1 1" />
+          </geometry>
+        </visual>
+        <!-- In rexrov2_base they made collision planes to minize the GPU load -->
+        <!-- <collision>
+          <origin xyz="0 0 0" rpy="0 0 0"/>
+          <geometry>
+            <mesh filename="${collision_mesh_file}" scale="1 1 1" />
+          </geometry>
+        </collision> -->
+      </link>
+    <gazebo reference="${namespace}/base_link">
+      <selfCollide>false</selfCollide>
+    </gazebo>
     <!-- Set up hydrodynamic plugin given as input parameter -->
     <xacro:insert_block name="gazebo"/>
-    <!-- optional: plugin to test compare Gazebo's returned accelerations
-    <gazebo>
-      <plugin name="${namespace}_test_plugin" filename="libaccelerations_test_plugin.so">
-        <link_name>${namespace}/base_link</link_name>
-      </plugin>
-    </gazebo> -->
    <!-- Publishes -->
    <!-- ONLY NEED FOR SIMULATIONS (GAZEBO SPECIFIC)

File: uuv_simulator/manta_description/urdf/manta_gazebo.xacro (robot description, xacro)
@@ -1,55 +1,83 @@
 <?xml version="1.0"?>
-<!-- Copyright (c) 2016 The UUV Simulator Authors.
-     All rights reserved.
-     Licensed under the Apache License, Version 2.0 (the "License");
-     you may not use this file except in compliance with the License.
-     You may obtain a copy of the License at
-       http://www.apache.org/licenses/LICENSE-2.0
-     Unless required by applicable law or agreed to in writing, software
-     distributed under the License is distributed on an "AS IS" BASIS,
-     WITHOUT WARRANTIES OR CONDITIONS OF ANY KIND, either express or implied.
-     See the License for the specific language governing permissions and
-     limitations under the License.
--->
 <robot xmlns:xacro="http://www.ros.org/wiki/xacro">
-    <!--
-    Center of buoyancy according to eq. (3.1) p. 28 in Berg2012.
-    The original values, [0.0822, -0.00773, 0.3872] however, seem to
-    assume NWU (otherwise cob is below cog?).
-    -->
-    <xacro:property name="cob" value="0.0 0.0 0.30"/>
-    <!-- Volume, see p.31 in Berg2012 -->
-    <xacro:property name="volume" value="1.820"/>
-    <xacro:macro name="manta_hydro_model" params="namespace">
-        <link name="${namespace}/base_link">
-            <neutrally_buoyant>0</neutrally_buoyant>
-            <volume>${volume}</volume>
-            <box>
-                <width>1.5</width>
-                <length>2.5</length>
-                <height>1.6</height>
-            </box>
-            <center_of_buoyancy>${cob}</center_of_buoyancy>
-            <hydrodynamic_model>
-                <type>fossen</type>
-                <!-- Added mass: see p.28 in Berg2012 -->
-                <added_mass>
-                     779.79 -6.8773 -103.32  8.5426 -165.54 -7.8033
-                    -6.8773    1222   51.29  409.44 -5.8488  62.726
-                    -103.32   51.29  3659.9  6.1112 -386.42  10.774
-                     8.5426  409.44  6.1112   534.9 -10.027  21.019
-                    -165.54 -5.8488 -386.42 -10.027  842.69 -1.1162
-                    -7.8033  62.726  10.775  21.019 -1.1162  224.32
-                </added_mass>
-                <!-- Linear damping: see p.31 in Berg2012 -->
-                <linear_damping>
-                    -74.82 -69.48 -728.4 -268.8 -309.77 -105
-                </linear_damping>
-                <!-- Non-linear damping: see p.30 in Berg2012 -->
-                <quadratic_damping>
-                    -748.22 -992.53 -1821.01 -672 -774.44 -523.27
-                </quadratic_damping>
-            </hydrodynamic_model>
-        </link>
-    </xacro:macro>
+  <xacro:macro name="manta_hydro_model" params="namespace">
+    <!-- List of hydrodynamic models this robot's links -->
+    <link name="${namespace}/base_link">
+      <!-- This flag will make the link neutrally buoyant -->
+      <neutrally_buoyant>0</neutrally_buoyant>
+      <!-- Link's volume -->
+      <volume>${volume}</volume>
+      <!-- Link's bounding box, it is used to recalculate the immersed
+        volume when close to the surface.
+        This is a workaround the invalid bounding box given by Gazebo-->
+      <box>
+        <width>${x_size}</width>
+        <length>${y_size}</length>
+        <height>${z_size}</height>
+      </box>
+      <!-- Center of buoyancy -->
+      <center_of_buoyancy>${cob}</center_of_buoyancy>
+      <!-- Fossen's equation of motion for underwater vehicles
+      Reference:
+          [1] Fossen, Thor I. Handbook of marine craft hydrodynamics and motion
+          control. John Wiley & Sons, 2011.
+     -->
+      <hydrodynamic_model>
+          <type>fossen</type>
+          <!-- Added mass: see p.28 in Berg2012 -->
+          <added_mass>
+            1.7182 0 0 0 0 0
+            0 0 0 0 0 0
+            0 0 5.468 0 0 0
+            0 0 0 10 0 0
+            0 0 0 0 10.2481 0
+            0 0 0 0 0 0.4006
+          </added_mass>
+          <!--
+            The linear damping coefficients can be provided as a diagonal (6 elements)
+            or a full matrix (36 coefficients), like the added-mass coefficients above
+            Linear damping: see p.31 in Berg2012
+          -->
+          <linear_damping>
+            -11.7391 -20 -31.8678 -25 -44.9085 -5
+          </linear_damping>
+          <!--
+            The linear damping coefficients proportional to the forward speed
+            can be provided as a diagonal (6 elements) or a full matrix (36 coefficients),
+            like the added-mass coefficients above.
+            This matrix is mostly useful for slender bodies (e.g. AUVs with torpedo shape)
+          -->
+          <!-- <linear_damping_forward_speed>
+            0 0 0 0 0 0
+          </linear_damping_forward_speed> -->
+          <!--
+            The quadratic damping coefficients can be provided as a diagonal (6 elements)
+            or a full matrix (36 coefficients), like the added-mass coefficients above
+            Non-linear damping: see p.30 in Berg2012
+          -->
+          <quadratic_damping>
+            0 0 0 0 0 0
+          </quadratic_damping>
+          <!--
+            In case you want to model a simple surface vessel, you can use the
+            implementation of linear (small angle) theory for boxed shaped vessels
+            by providing the following parameters. If you omit the area of the
+            water level plane area, it will be calculated from the bounding box
+            parameters. Uncomment the lines below in case you are simulating a
+            surface vessel.
+            For more details on these parameters and the computation of buoyancy
+            for vessels using this theory, check:
+              [1] Lecture Notes  TTK 4190 Guidance and Control of Vehicles (T. I. Fossen)
+                  http://www.fossen.biz/wiley/Ch4.pdf
+              [2] Fossen, Thor I. Handbook of marine craft hydrodynamics and motion
+                  control. John Wiley & Sons, 2011.
+          -->
+          <!--
+          <metacentric_width>0.0</metacentric_width>
+          <metacentric_length>0.0</metacentric_length>
+          <water_level_plane_area>0.0</water_level_plane_area>
+          -->
+      </hydrodynamic_model>
+    </link>
+  </xacro:macro>
 </robot>

Commit message: changed the hydrodynamics and thruster dynamics of Manta

File: uuv_simulator/manta_description/urdf/manta_actuators.xacro (robot description, xacro)
@@ -17,6 +17,6 @@
       thruster_id="${thruster_id}"
       mesh_filename="${prop_mesh_file_cw}"
-      dyn_time_constant="0.05"
-      rotor_constant="1.0">
+      dyn_time_constant="0.4"
+      rotor_constant="0.000004">
       <xacro:insert_block name="origin"/>
     </xacro:thruster_module_first_order_basic_fcn_macro>
@@ -28,6 +28,6 @@
       thruster_id="${thruster_id}"
       mesh_filename="${prop_mesh_file_ccw}"
-      dyn_time_constant="0.05"
-      rotor_constant="1.0">
+      dyn_time_constant="0.4"
+      rotor_constant="0.000004">
       <xacro:insert_block name="origin"/>
     </xacro:thruster_module_first_order_basic_fcn_macro>

File: uuv_simulator/manta_description/urdf/manta_base.xacro (robot description, xacro)
@@ -22,5 +22,5 @@
   -->
   <!-- Mass -->
-  <xacro:property name="mass" value="19.0"/>
+  <xacro:property name="mass" value="16.6"/>
   <!-- Describing the dimensions of the vehicle's bounding box: width, length, height -->
   <xacro:property name="x_size" value="0.448"/>
@@ -31,5 +31,5 @@
   <xacro:property name="volume" value="0.01854"/>
   <!-- Center of gravity -->
-  <xacro:property name="cog" value="0 0 -0.03"/>
+  <xacro:property name="cog" value="0 0 -0.08"/>
   <!--
   Center of buoyancy according to eq. (3.1) p. 28 in Berg2012.
@@ -59,6 +59,4 @@
           <mass value="${mass}" />
           <origin xyz="${cog}" rpy="0 0 0"/>
-           <!-- ixx="${0.80947}" ixy="-0.00308" ixz="-0.01546"
-            iyy="${0.87794}" iyz="0.06283" izz="${1.57147}" />  -->
           <inertia
             ixx="${0.503217}" ixy="${0.000204}" ixz="${-0.000526}"

File: uuv_simulator/manta_description/urdf/manta_gazebo.xacro (robot description, xacro)
@@ -31,10 +31,10 @@
           <!-- Added mass: see p.28 in Berg2012 -->
           <added_mass>
-            1.7182 0 0 0 0 0
-            0 0 0 0 0 0
-            0 0 5.468 0 0 0
-            0 0 0 10 0 0
-            0 0 0 0 10.2481 0
-            0 0 0 0 0 0.4006
+            10.7727 0 0 0 0 0
+            0 10.7727 0 0 0 0
+            0 0 49.7679 0 0 0
+            0 0 0 1.0092 0 0
+            0 0 0 0 1.0092 0
+            0  0  0  0  0  0
           </added_mass>
           <!--
@@ -44,5 +44,5 @@
           -->
           <linear_damping>
-            -11.7391 -20 -31.8678 -25 -44.9085 -5
+            -9.5909 -9.5909 -42.5798 -13.3040 -13.2181 -1.1559
           </linear_damping>
           <!--
@@ -61,5 +61,5 @@
           -->
           <quadratic_damping>
-            0 0 0 0 0 0
+            -5.1386 -5.1386 -26.1105 0 0 0
           </quadratic_damping>
           <!--

File: uuv_simulator/uuv_gazebo_plugins/uuv_gazebo_ros_plugins/urdf/thruster_snippets.xacro (robot description, xacro)
@@ -83,5 +83,5 @@
     </joint>
     <link name="${namespace}/thruster_${thruster_id}">
-      <xacro:box_inertial x="0" y="0" z="0" mass="0.001">
+      <xacro:box_inertial x="0.3" y="0.3" z="0.3" mass="0.3">
         <origin xyz="0 0 0" rpy="0 0 0"/>
       </xacro:box_inertial>
