Commit message: gripper, configurable dynamic shoulder, drone prefix

File: auv_setup/description/drone.urdf.xacro (robot description, xacro)
@@ -3,4 +3,5 @@
   <xacro:arg name="include_flir" default="false"/>
   <xacro:arg name="include_gripper" default="false"/>
+  <xacro:arg name="static_shoulder" default="true"/>
   <link name="base_link"></link>
   <link name="imu_link"></link>
@@ -8,4 +9,6 @@
   <link name="pressure_sensor_link"></link>
   <link name="sonar_link"></link>
+  <link name="front_camera_link"/>
+  <link name="downwards_camera_link"/>
   <!-- base to imu -->
   <joint name="base_to_imu" type="fixed">
@@ -33,14 +36,15 @@
   </joint>
   <xacro:if value="$(arg include_flir)">
-    <!-- Prefer local lightweight FLIR links helper when available. This
-         avoids pulling in the full flir_camera_description package which
-         may be absent in some workspaces. -->
-  <xacro:include filename="flir_blackfly_s.urdf.xacro"/>
-    <xacro:flir_blackfly_s parent="base_link" frame="flir_camera_link" name="flir_blackfly">
+    <xacro:include filename="flir_blackfly_s.urdf.xacro"/>
+    <joint name="base_to_downwards_camera" type="fixed">
+      <parent link="base_link"/>
+      <child link="downwards_camera_link"/>
       <origin xyz="0.283615 -0.085021 0.094186" rpy="0.0 0 1.5708"/>
-    </xacro:flir_blackfly_s>
+    </joint>
+  <xacro:flir_blackfly_s frame="downwards_camera_link" base="downwards_camera" name="flir_blackfly"/>
   </xacro:if>
   <xacro:if value="$(arg include_gripper)">
-    <xacro:include filename="$(find gripper_description)/urdf/gripper.urdf.xacro"/>
+    <xacro:include filename="gripper.urdf.xacro"/>
+    <link name="gripper_link"/>
     <joint name="base_to_gripper" type="fixed">
       <parent link="base_link"/>
@@ -48,9 +52,13 @@
       <origin xyz="0.26 0.095 0.08" rpy="0 0 0"/>
     </joint>
+    <xacro:gripper frame="gripper_link" static_shoulder="$(arg static_shoulder)"/>
   </xacro:if>
   <!-- RealSense -->
   <xacro:include filename="realsense_d555.urdf.xacro"/>
-  <xacro:realsense_d555 parent="base_link" frame="realsense" name="realsense">
+  <joint name="base_to_front_camera" type="fixed">
+    <parent link="base_link"/>
+    <child link="front_camera_link"/>
     <origin xyz="0.36362 0.0 -0.023395" rpy="3.14159 0 0"/>
-  </xacro:realsense_d555>
+  </joint>
+  <xacro:realsense_d555 frame="front_camera_link" base="front_camera" name="realsense"/>
 </robot>

File: auv_setup/description/flir_blackfly_s.urdf.xacro (robot description, xacro)
@@ -6,32 +6,35 @@
     collisions, inertial and Gazebo sensor/plugin blocks so it can be
     included in robot descriptions when only TF frames are required.
-    Usage (similar to realsense helper):
+    The caller is responsible for declaring ${frame} as a <link> and
+    connecting it to the parent with a <joint> (+ the desired origin).
+    This macro only adds the sensor sub-frames below ${frame}.
+    Usage:
       <xacro:include filename="flir_blackfly_s.urdf.xacro"/>
-      <xacro:flir_blackfly_s parent="base_link" name="realsense" frame="flir_camera"/>
+      <link name="downwards_camera_link"/>
+      <joint name="base_to_downwards_camera" type="fixed">
+        <parent link="base_link"/>
+        <child link="downwards_camera_link"/>
+        <origin xyz="0.28 -0.08 0.09" rpy="0 0 1.5708"/>
+      </joint>
+      <xacro:flir_blackfly_s frame="downwards_camera_link" name="flir_blackfly"/>
   -->
-  <xacro:macro name="flir_blackfly_s" params="parent *origin frame:=camera name:=camera lens_h:=0.04">
-    <!-- Mount joint: attach the camera base link to the given parent -->
-    <joint name="${frame}_mount_joint" type="fixed">
-      <xacro:insert_block name="origin"/>
-      <parent link="${parent}"/>
-      <child link="${frame}"/>
-    </joint>
-    <!-- Camera body link (minimal) -->
-    <link name="${frame}"/>
+  <xacro:macro name="flir_blackfly_s" params="frame base name:=camera lens_h:=0.04">
+    <!-- 'base' must be provided by the caller and should be the desired
+         prefix for generated sub-frame names (e.g. 'downwards_camera'). -->
     <!-- Lens and optical links (minimal) -->
-    <link name="${frame}_lens"/>
-    <link name="${frame}_optical"/>
+    <link name="${base}_lens"/>
+    <link name="${base}_optical"/>
     <!-- Fixed joint from body to lens (keeps original relative origin) -->
-    <joint name="${frame}_lens_joint" type="fixed">
+    <joint name="${base}_lens_joint" type="fixed">
       <!-- origin taken from flir_blackfly_s xacro: 0.02685 0 0.01425 -->
       <origin xyz="0.02685 0 0.01425" rpy="0 0 0"/>
       <parent link="${frame}"/>
-      <child link="${frame}_lens"/>
+      <child link="${base}_lens"/>
     </joint>
     <!-- Fixed joint from lens to optical frame. Lens length is parameterized. -->
-    <joint name="${frame}_optical_joint" type="fixed">
+    <joint name="${base}_optical_joint" type="fixed">
       <origin xyz="${lens_h} 0 0" rpy="-1.570796 0 -1.570796"/>
-      <parent link="${frame}_lens"/>
-      <child link="${frame}_optical"/>
+      <parent link="${base}_lens"/>
+      <child link="${base}_optical"/>
     </joint>
   </xacro:macro>

File: auv_setup/description/realsense_d555.urdf.xacro (robot description, xacro)
@@ -13,5 +13,5 @@
     to depth-frame values need to be updated.
   -->
-  <xacro:macro name="realsense_d555" params="parent *origin name:=camera frame:=camera">
+  <xacro:macro name="realsense_d555" params="frame base name:=camera">
     <xacro:property name="M_PI" value="3.1415926535897931" />
     <!-- Mount-hole -> depth/infra1 frame offsets (default: D455-style) -->
@@ -23,63 +23,63 @@
     <xacro:property name="depth_to_infra2_y" value="-0.095" />
     <xacro:property name="depth_to_color_y"  value="-0.059" />
-    <!-- Mount/screw-hole frame -->
-    <joint name="${name}_mount_joint" type="fixed">
-      <xacro:insert_block name="origin" />
-      <parent link="${parent}"/>
-      <child link="${frame}_link"/>
-    </joint>
-    <link name="${frame}_link"/>
+    <!-- 'base' must be provided by the caller and should be the desired
+         prefix for generated sub-frame names (e.g. 'front_camera'). -->
+    <!--
+      The caller is responsible for declaring ${frame} as a <link> and
+      connecting it to the parent with a <joint> (+ the desired origin).
+      This macro only adds the sensor sub-frames below ${frame}.
+    -->
     <!-- Depth frame (same nominal origin as infra1 in the D455 xacro) -->
     <joint name="${name}_depth_joint" type="fixed">
       <origin xyz="${depth_px} ${depth_py} ${depth_pz}" rpy="0 0 0"/>
-      <parent link="${frame}_link"/>
-      <child link="${frame}_depth_frame"/>
+      <parent link="${frame}"/>
+      <child link="${base}_depth"/>
     </joint>
-    <link name="${frame}_depth_frame"/>
+    <link name="${base}_depth"/>
     <joint name="${name}_depth_optical_joint" type="fixed">
       <origin xyz="0 0 0" rpy="${-M_PI/2} 0 ${-M_PI/2}"/>
-      <parent link="${frame}_depth_frame"/>
-      <child link="${frame}_depth_optical_frame"/>
+      <parent link="${base}_depth"/>
+      <child link="${base}_depth_optical"/>
     </joint>
-    <link name="${frame}_depth_optical_frame"/>
+    <link name="${base}_depth_optical"/>
     <!-- Infrared 1 frame -->
     <joint name="${name}_infra1_joint" type="fixed">
       <origin xyz="${depth_px} ${depth_py + depth_to_infra1_y} ${depth_pz}" rpy="0 0 0"/>
-      <parent link="${frame}_link"/>
-      <child link="${frame}_infra1_frame"/>
+      <parent link="${frame}"/>
+      <child link="${base}_infra1"/>
     </joint>
-    <link name="${frame}_infra1_frame"/>
+    <link name="${base}_infra1"/>
     <joint name="${name}_infra1_optical_joint" type="fixed">
       <origin xyz="0 0 0" rpy="${-M_PI/2} 0 ${-M_PI/2}"/>
-      <parent link="${frame}_infra1_frame"/>
-      <child link="${frame}_infra1_optical_frame"/>
+      <parent link="${base}_infra1"/>
+      <child link="${base}_infra1_optical"/>
     </joint>
-    <link name="${frame}_infra1_optical_frame"/>
+    <link name="${base}_infra1_optical"/>
     <!-- Infrared 2 frame -->
     <joint name="${name}_infra2_joint" type="fixed">
       <origin xyz="${depth_px} ${depth_py + depth_to_infra2_y} ${depth_pz}" rpy="0 0 0"/>
-      <parent link="${frame}_link"/>
-      <child link="${frame}_infra2_frame"/>
+      <parent link="${frame}"/>
+      <child link="${base}_infra2"/>
     </joint>
-    <link name="${frame}_infra2_frame"/>
+    <link name="${base}_infra2"/>
     <joint name="${name}_infra2_optical_joint" type="fixed">
       <origin xyz="0 0 0" rpy="${-M_PI/2} 0 ${-M_PI/2}"/>
-      <parent link="${frame}_infra2_frame"/>
-      <child link="${frame}_infra2_optical_frame"/>
+      <parent link="${base}_infra2"/>
+      <child link="${base}_infra2_optical"/>
     </joint>
-    <link name="${frame}_infra2_optical_frame"/>
+    <link name="${base}_infra2_optical"/>
     <!-- Color frame -->
     <joint name="${name}_color_joint" type="fixed">
       <origin xyz="${depth_px} ${depth_py + depth_to_color_y} ${depth_pz}" rpy="0 0 0"/>
-      <parent link="${frame}_link"/>
-      <child link="${frame}_color_frame"/>
+      <parent link="${frame}"/>
+      <child link="${base}_color"/>
     </joint>
-    <link name="${frame}_color_frame"/>
+    <link name="${base}_color"/>
     <joint name="${name}_color_optical_joint" type="fixed">
       <origin xyz="0 0 0" rpy="${-M_PI/2} 0 ${-M_PI/2}"/>
-      <parent link="${frame}_color_frame"/>
-      <child link="${frame}_color_optical_frame"/>
+      <parent link="${base}_color"/>
+      <child link="${base}_color_optical"/>
     </joint>
-    <link name="${frame}_color_optical_frame"/>
+    <link name="${base}_color_optical"/>
   </xacro:macro>
 </robot>
