Commit message: urdf for orca + moby

File: auv_setup/description/moby.urdf.xacro (robot description, xacro)
@@ -1,7 +1,4 @@
 <?xml version="1.0"?>
 <robot name="orca" xmlns:xacro="http://ros.org/wiki/xacro">
-  <xacro:arg name="include_flir" default="false"/>
-  <xacro:arg name="include_gripper" default="false"/>
-  <xacro:arg name="static_shoulder" default="true"/>
   <link name="base_link"></link>
   <link name="imu_link"></link>
@@ -11,5 +8,5 @@
   <link name="front_camera_link"/>
   <link name="downwards_camera_link"/>
-  <!-- base to imu -->
+  <!-- base to imu. NB! Needs updated position once mounted on drone! -->
   <joint name="base_to_imu" type="fixed">
     <parent link="base_link"/>
@@ -35,23 +32,20 @@
     <origin xyz="0.271721 0.0 -0.203397" rpy="0.0 0.0 0.0"/>
   </joint>
-  <xacro:if value="$(arg include_flir)">
-    <xacro:include filename="flir_blackfly_s.urdf.xacro"/>
-    <joint name="base_to_downwards_camera" type="fixed">
-      <parent link="base_link"/>
-      <child link="downwards_camera_link"/>
-      <origin xyz="0.283615 -0.085021 0.094186" rpy="0.0 0 1.5708"/>
-    </joint>
+  <xacro:include filename="flir_blackfly_s.urdf.xacro"/>
+  <joint name="base_to_downwards_camera" type="fixed">
+    <parent link="base_link"/>
+    <child link="downwards_camera_link"/>
+    <origin xyz="0.283615 -0.085021 0.094186" rpy="-1.5708 -1.5708 -1.5708"/>
+  </joint>
   <xacro:flir_blackfly_s frame="downwards_camera_link" base="downwards_camera" name="flir_blackfly"/>
-  </xacro:if>
-  <xacro:if value="$(arg include_gripper)">
-    <xacro:include filename="gripper.urdf.xacro"/>
-    <link name="gripper_link"/>
-    <joint name="base_to_gripper" type="fixed">
-      <parent link="base_link"/>
-      <child link="gripper_link"/>
-      <origin xyz="0.26 0.095 0.08" rpy="0 0 0"/>
-    </joint>
-    <xacro:gripper frame="gripper_link" static_shoulder="$(arg static_shoulder)"/>
-  </xacro:if>
+  <xacro:include filename="gripper.urdf.xacro"/>
+  <!-- Gripper needs updated urdf with the new model once ready-->
+  <link name="gripper_link"/>
+  <joint name="base_to_gripper" type="fixed">
+    <parent link="base_link"/>
+    <child link="gripper_link"/>
+    <origin xyz="0.26 0.095 0.08" rpy="0 0 0"/>
+  </joint>
+  <xacro:gripper frame="gripper_link" static_shoulder="true"/>
   <!-- RealSense -->
   <xacro:include filename="realsense_d555.urdf.xacro"/>

Commit message: added gripper urdf for moby

File: auv_setup/description/moby.urdf.xacro (robot description, xacro)
@@ -39,13 +39,4 @@
   </joint>
   <xacro:flir_blackfly_s frame="downwards_camera_link" base="downwards_camera" name="flir_blackfly"/>
-  <xacro:include filename="gripper.urdf.xacro"/>
-  <!-- Gripper needs updated urdf with the new model once ready-->
-  <link name="gripper_link"/>
-  <joint name="base_to_gripper" type="fixed">
-    <parent link="base_link"/>
-    <child link="gripper_link"/>
-    <origin xyz="0.26 0.095 0.08" rpy="0 0 0"/>
-  </joint>
-  <xacro:gripper frame="gripper_link" static_shoulder="true"/>
   <!-- RealSense -->
   <xacro:include filename="realsense_d555.urdf.xacro"/>
@@ -56,3 +47,34 @@
   </joint>
   <xacro:realsense_d555 frame="front_camera_link" base="front_camera" name="realsense"/>
+  <!-- Gripper -->
+  <link name="shoulder"></link>
+  <joint name="shoulder_joint" type="fixed">
+    <parent link="base_link"/>
+    <child link="shoulder"/>
+    <origin xyz="0.282589 0.07822 0.115803" rpy="0.0 0.0 0.0"/>
+  </joint>
+  <link name="arm"></link>
+  <joint name="moby/arm_joint" type="revolute">
+    <parent link="shoulder"/>
+    <child link="arm"/>
+    <origin xyz="0.0 0.0 0.0" rpy="0.0 0.0 0.0"/>
+    <axis xyz="1.0 0.0 0.0"/>
+    <limit lower="-3.14159" upper="3.14159" effort="0" velocity="0"/>
+  </joint>
+  <link name="finger1"></link>
+  <joint name="moby/finger_joint1" type="prismatic">
+    <parent link="arm"/>
+    <child link="finger1"/>
+    <origin xyz="0.0 0.0 0.0" rpy="0.0 0.0 0.0"/>
+    <axis xyz="0.70711 0.70711 0.0"/>
+    <limit lower="-0.033" upper="0" effort="0" velocity="0"/>
+  </joint>
+  <link name="finger2"></link>
+  <joint name="moby/finger_joint2" type="prismatic">
+    <parent link="arm"/>
+    <child link="finger2"/>
+    <origin xyz="0.0 0.0 0.0" rpy="0.0 0.0 0.0"/>
+    <axis xyz="0.70711 -0.70711 0.0"/>
+    <limit lower="-0.033" upper="0" effort="0" velocity="0"/>
+  </joint>
 </robot>
