Commit message: rename new drone

File: auv_setup/description/nautilus.urdf.xacro (robot description, xacro)
@@ -55,5 +55,5 @@
   </joint>
   <link name="arm"></link>
-  <joint name="moby/arm_joint" type="revolute">
+  <joint name="nautilus/arm_joint" type="revolute">
     <parent link="shoulder"/>
     <child link="arm"/>
@@ -63,5 +63,5 @@
   </joint>
   <link name="finger1"></link>
-  <joint name="moby/finger_joint1" type="prismatic">
+  <joint name="nautilus/finger_joint1" type="prismatic">
     <parent link="arm"/>
     <child link="finger1"/>
@@ -71,5 +71,5 @@
   </joint>
   <link name="finger2"></link>
-  <joint name="moby/finger_joint2" type="prismatic">
+  <joint name="nautilus/finger_joint2" type="prismatic">
     <parent link="arm"/>
     <child link="finger2"/>

Commit message: update imu tf

File: auv_setup/description/nautilus.urdf.xacro (robot description, xacro)
@@ -12,5 +12,5 @@
     <parent link="base_link"/>
     <child link="imu_link"/>
-    <origin xyz="0.0057 0.0 0.0827" rpy="0.0 0.0 0.0"/>
+    <origin xyz="-0.1 -0.001 0.085" rpy="0.0 0.0 0.0"/>
   </joint>
   <!-- base to dvl -->

Commit message: urfd: updated gripper position

File: auv_setup/description/nautilus.urdf.xacro (robot description, xacro)
@@ -52,5 +52,5 @@
     <parent link="base_link"/>
     <child link="shoulder"/>
-    <origin xyz="0.282589 0.07822 0.115803" rpy="0.0 0.0 0.0"/>
+    <origin xyz="0.282589 0.028 0.115803" rpy="0.0 0.0 0.0"/>
   </joint>
   <link name="arm"></link>

Commit message: URDF: update down cam link

File: auv_setup/description/nautilus.urdf.xacro (robot description, xacro)
@@ -36,5 +36,5 @@
     <parent link="base_link"/>
     <child link="downwards_camera_link"/>
-    <origin xyz="0.283615 -0.085021 0.094186" rpy="-1.5708 -1.5708 -1.5708"/>
+    <origin xyz="0.283615 -0.158 0.094186" rpy="-1.5708 -1.5708 -1.5708"/>
   </joint>
   <xacro:flir_blackfly_s frame="downwards_camera_link" base="downwards_camera" name="flir_blackfly"/>

Commit message: tf: move down cam down

File: auv_setup/description/nautilus.urdf.xacro (robot description, xacro)
@@ -36,5 +36,5 @@
     <parent link="base_link"/>
     <child link="downwards_camera_link"/>
-    <origin xyz="0.283615 -0.158 0.094186" rpy="-1.5708 -1.5708 -1.5708"/>
+    <origin xyz="0.283615 -0.158 0.12" rpy="-1.5708 -1.5708 -1.5708"/>
   </joint>
   <xacro:flir_blackfly_s frame="downwards_camera_link" base="downwards_camera" name="flir_blackfly"/>

Commit message: Added ins origin logic. Rotated tf2 dvl frame

File: auv_setup/description/nautilus.urdf.xacro (robot description, xacro)
@@ -18,5 +18,5 @@
     <parent link="base_link"/>
     <child link="dvl_link"/>
-    <origin xyz="-0.130 0.003 0.2414" rpy="0.0 0.0 0.0"/>
+    <origin xyz="-0.130 0.003 0.2414" rpy="0.0 0.0 3.14159"/>
   </joint>
   <!-- base to pressure sensor -->

Commit message: added reset service call for landmark, referencefilter, waypointmanager

File: auv_setup/description/nautilus.urdf.xacro (robot description, xacro)
@@ -78,3 +78,10 @@
     <limit lower="-0.033" upper="0" effort="0" velocity="0"/>
   </joint>
+  <!-- Virtual reference frame at the centre of the gripper jaw opening -->
+  <link name="grip_point"></link>
+  <joint name="grip_point_joint" type="fixed">
+    <parent link="shoulder"/>
+    <child link="grip_point"/>
+    <origin xyz="0.2505 0.0 0.0" rpy="0.0 0.0 0.0"/>
+  </joint>
 </robot>

Commit message: update naut pressure tf

File: auv_setup/description/nautilus.urdf.xacro (robot description, xacro)
@@ -24,5 +24,5 @@
     <parent link="base_link"/>
     <child link="pressure_sensor_link"/>
-    <origin xyz="-0.130 0.003 0.2414" rpy="0.0 0.0 0.0"/>
+    <origin xyz="-0.035 -0.115 -0.095" rpy="0.0 0.0 0.0"/>
   </joint>
   <!-- base to fls -->

Commit message: jørgen changes

File: auv_setup/description/nautilus.urdf.xacro (robot description, xacro)
@@ -44,5 +44,5 @@
     <parent link="base_link"/>
     <child link="front_camera_link"/>
-    <origin xyz="0.36362 0.0 -0.023395" rpy="3.14159 0 0"/>
+    <origin xyz="0.36362 0.0 -0.023395" rpy="3.14159 -0.261666667 0"/>
   </joint>
   <xacro:realsense_d555 frame="front_camera_link" base="front_camera" name="realsense"/>
