Commit message: nautilus: front camera is level, not pitched 15 deg down
The 15 deg pitch on base_to_front_camera does not match the real
camera or the simulator (nautilus.scn), so every slalom pole was put
1.4-1.7 m too deep and ~10 % too close in the sim.

Co-Authored-By: Claude Opus 5.5 <noreply@anthropic.com>

File: auv_setup/description/nautilus.urdf.xacro (robot description, xacro)
@@ -44,5 +44,5 @@
     <parent link="base_link"/>
     <child link="front_camera_link"/>
-    <origin xyz="0.36362 0.0 -0.023395" rpy="3.14159 -0.261666667 0"/>
+    <origin xyz="0.36362 0.0 -0.023395" rpy="3.14159 0 0"/>
   </joint>
   <xacro:realsense_d555 frame="front_camera_link" base="front_camera" name="realsense"/>
